Commit message: update urdf joint limits

File: src/simple_assembly/urdf/simple_assembly.urdf (robot description, URDF)
Before this commit: robot simple_assembly, 17 links, 16 joints
Joints:
- joint revolute_1_0: limit lower=-1.9199 upper=1.9199 effort=150.0 velocity=15.71 -> lower=-6.28318 upper=6.28318 effort=150.0 velocity=15.71
- joint revolute_2_0: limit lower=-3.14159 upper=3.14159 effort=27.0 velocity=5.45 -> lower=-1.5708 upper=1.5708 effort=27.0 velocity=5.45
- joint revolute_3_0: limit lower=-1.9199 upper=1.9199 effort=150.0 velocity=15.71 -> lower=-6.28318 upper=6.28318 effort=150.0 velocity=15.71
- joint revolute_4_0: limit lower=-3.14159 upper=3.14159 effort=27.0 velocity=5.45 -> lower=-1.91986 upper=1.91986 effort=27.0 velocity=5.45
- joint revolute_5_0: limit lower=-1.9199 upper=1.9199 effort=150.0 velocity=15.71 -> lower=-6.28318 upper=6.28318 effort=150.0 velocity=15.71
- joint revolute_6_0: limit lower=-3.14159 upper=3.14159 effort=27.0 velocity=5.45 -> lower=-1.91986 upper=1.91986 effort=27.0 velocity=5.45
- joint revolute_7_0: limit lower=-1.9199 upper=1.9199 effort=150.0 velocity=15.71 -> lower=-6.28318 upper=6.28318 effort=150.0 velocity=15.71
