Commit message: Add ROS-backed kiosk web interface simulation stack

File: src/simple_assembly_moveit_config/config/simple_assembly.ros2_control.xacro (robot description, xacro)
@@ -1,11 +1,16 @@
 <?xml version="1.0"?>
 <robot xmlns:xacro="http://www.ros.org/wiki/xacro">
-    <xacro:macro name="simple_assembly_ros2_control" params="name">
+    <xacro:macro name="simple_assembly_ros2_control" params="name use_fake_hardware:=false">
         <ros2_control name="${name}" type="system">
             <hardware>
-                <plugin>damiao_driver/DamiaoHardwareInterface</plugin>
-                <param name="serial_port">/dev/ttyACM0</param>
-                <param name="baud_rate">921600</param>
-                <param name="control_mode">position</param>
+                <xacro:if value="${use_fake_hardware}">
+                    <plugin>mock_components/GenericSystem</plugin>
+                </xacro:if>
+                <xacro:unless value="${use_fake_hardware}">
+                    <plugin>damiao_driver/DamiaoHardwareInterface</plugin>
+                    <param name="serial_port">/dev/ttyACM0</param>
+                    <param name="baud_rate">921600</param>
+                    <param name="control_mode">position</param>
+                </xacro:unless>
             </hardware>
             <!-- Joint 1 (base): Z-type DM10010, physical top-to-bottom index 7 -->

File: src/simple_assembly_moveit_config/config/simple_assembly.urdf.xacro (robot description, xacro)
@@ -1,8 +1,12 @@
 <?xml version="1.0"?>
 <robot xmlns:xacro="http://www.ros.org/wiki/xacro" name="simple_assembly">
+    <xacro:arg name="use_fake_hardware" default="false" />
     <!-- Import simple_assembly urdf file -->
     <xacro:include filename="$(find simple_assembly)/urdf/simple_assembly.urdf" />
     <!-- Import control_xacro -->
     <xacro:include filename="simple_assembly.ros2_control.xacro" />
-    <xacro:simple_assembly_ros2_control name="DamiaoArm"/>
+    <xacro:simple_assembly_ros2_control
+        name="DamiaoArm"
+        use_fake_hardware="$(arg use_fake_hardware)"
+    />
 </robot>

Commit message: Persist Damiao zero offsets

File: src/simple_assembly_moveit_config/config/simple_assembly.ros2_control.xacro (robot description, xacro)
@@ -1,5 +1,5 @@
 <?xml version="1.0"?>
 <robot xmlns:xacro="http://www.ros.org/wiki/xacro">
-    <xacro:macro name="simple_assembly_ros2_control" params="name">
+    <xacro:macro name="simple_assembly_ros2_control" params="name calibrate_on_start:=false zero_offsets_file:=/home/terralabscove/.ros/damiao_zero_offsets.yaml">
         <ros2_control name="${name}" type="system">
             <hardware>
@@ -8,4 +8,6 @@
                 <param name="baud_rate">921600</param>
                 <param name="control_mode">position</param>
+                <param name="zero_offsets_file">${zero_offsets_file}</param>
+                <param name="calibrate_on_start">${calibrate_on_start}</param>
             </hardware>
             <!-- Joint 1 (base): Z-type DM10010, physical top-to-bottom index 7 -->

File: src/simple_assembly_moveit_config/config/simple_assembly.urdf.xacro (robot description, xacro)
@@ -5,4 +5,9 @@
     <!-- Import control_xacro -->
     <xacro:include filename="simple_assembly.ros2_control.xacro" />
-    <xacro:simple_assembly_ros2_control name="DamiaoArm"/>
+    <xacro:arg name="calibrate_on_start" default="false"/>
+    <xacro:arg name="zero_offsets_file" default="/home/terralabscove/.ros/damiao_zero_offsets.yaml"/>
+    <xacro:simple_assembly_ros2_control
+        name="DamiaoArm"
+        calibrate_on_start="$(arg calibrate_on_start)"
+        zero_offsets_file="$(arg zero_offsets_file)"/>
 </robot>

File: src/simple_assembly_tracking_moveit_config/config/simple_assembly_tracking.ros2_control.xacro (robot description, xacro)
@@ -1,5 +1,5 @@
 <?xml version="1.0"?>
 <robot xmlns:xacro="http://www.ros.org/wiki/xacro">
-    <xacro:macro name="simple_assembly_tracking_ros2_control" params="name">
+    <xacro:macro name="simple_assembly_tracking_ros2_control" params="name calibrate_on_start:=false zero_offsets_file:=/home/terralabscove/.ros/damiao_zero_offsets.yaml">
         <ros2_control name="${name}" type="system">
             <hardware>
@@ -8,4 +8,6 @@
                 <param name="baud_rate">921600</param>
                 <param name="control_mode">position</param>
+                <param name="zero_offsets_file">${zero_offsets_file}</param>
+                <param name="calibrate_on_start">${calibrate_on_start}</param>
             </hardware>
             <!-- Joint 1 (base): Z-type DM10010, physical top-to-bottom index 7 -->

File: src/simple_assembly_tracking_moveit_config/config/simple_assembly_tracking.urdf.xacro (robot description, xacro)
@@ -2,5 +2,10 @@
 <robot xmlns:xacro="http://www.ros.org/wiki/xacro" name="simple_assembly_tracking">
     <xacro:include filename="$(find simple_assembly_tracking)/urdf/simple_assembly_tracking.urdf.xacro" />
+    <xacro:arg name="calibrate_on_start" default="false"/>
+    <xacro:arg name="zero_offsets_file" default="/home/terralabscove/.ros/damiao_zero_offsets.yaml"/>
     <xacro:include filename="simple_assembly_tracking.ros2_control.xacro" />
-    <xacro:simple_assembly_tracking_ros2_control name="DamiaoArm"/>
+    <xacro:simple_assembly_tracking_ros2_control
+        name="DamiaoArm"
+        calibrate_on_start="$(arg calibrate_on_start)"
+        zero_offsets_file="$(arg zero_offsets_file)"/>
 </robot>

Commit message: Revert Damiao zero offset persistence

File: src/simple_assembly_moveit_config/config/simple_assembly.ros2_control.xacro (robot description, xacro)
@@ -1,5 +1,5 @@
 <?xml version="1.0"?>
 <robot xmlns:xacro="http://www.ros.org/wiki/xacro">
-    <xacro:macro name="simple_assembly_ros2_control" params="name calibrate_on_start:=false zero_offsets_file:=/home/terralabscove/.ros/damiao_zero_offsets.yaml">
+    <xacro:macro name="simple_assembly_ros2_control" params="name">
         <ros2_control name="${name}" type="system">
             <hardware>
@@ -8,6 +8,4 @@
                 <param name="baud_rate">921600</param>
                 <param name="control_mode">position</param>
-                <param name="zero_offsets_file">${zero_offsets_file}</param>
-                <param name="calibrate_on_start">${calibrate_on_start}</param>
             </hardware>
             <!-- Joint 1 (base): Z-type DM10010, physical top-to-bottom index 7 -->

File: src/simple_assembly_moveit_config/config/simple_assembly.urdf.xacro (robot description, xacro)
@@ -5,9 +5,4 @@
     <!-- Import control_xacro -->
     <xacro:include filename="simple_assembly.ros2_control.xacro" />
-    <xacro:arg name="calibrate_on_start" default="false"/>
-    <xacro:arg name="zero_offsets_file" default="/home/terralabscove/.ros/damiao_zero_offsets.yaml"/>
-    <xacro:simple_assembly_ros2_control
-        name="DamiaoArm"
-        calibrate_on_start="$(arg calibrate_on_start)"
-        zero_offsets_file="$(arg zero_offsets_file)"/>
+    <xacro:simple_assembly_ros2_control name="DamiaoArm"/>
 </robot>

File: src/simple_assembly_tracking_moveit_config/config/simple_assembly_tracking.ros2_control.xacro (robot description, xacro)
@@ -1,5 +1,5 @@
 <?xml version="1.0"?>
 <robot xmlns:xacro="http://www.ros.org/wiki/xacro">
-    <xacro:macro name="simple_assembly_tracking_ros2_control" params="name calibrate_on_start:=false zero_offsets_file:=/home/terralabscove/.ros/damiao_zero_offsets.yaml">
+    <xacro:macro name="simple_assembly_tracking_ros2_control" params="name">
         <ros2_control name="${name}" type="system">
             <hardware>
@@ -8,6 +8,4 @@
                 <param name="baud_rate">921600</param>
                 <param name="control_mode">position</param>
-                <param name="zero_offsets_file">${zero_offsets_file}</param>
-                <param name="calibrate_on_start">${calibrate_on_start}</param>
             </hardware>
             <!-- Joint 1 (base): Z-type DM10010, physical top-to-bottom index 7 -->

File: src/simple_assembly_tracking_moveit_config/config/simple_assembly_tracking.urdf.xacro (robot description, xacro)
@@ -2,10 +2,5 @@
 <robot xmlns:xacro="http://www.ros.org/wiki/xacro" name="simple_assembly_tracking">
     <xacro:include filename="$(find simple_assembly_tracking)/urdf/simple_assembly_tracking.urdf.xacro" />
-    <xacro:arg name="calibrate_on_start" default="false"/>
-    <xacro:arg name="zero_offsets_file" default="/home/terralabscove/.ros/damiao_zero_offsets.yaml"/>
     <xacro:include filename="simple_assembly_tracking.ros2_control.xacro" />
-    <xacro:simple_assembly_tracking_ros2_control
-        name="DamiaoArm"
-        calibrate_on_start="$(arg calibrate_on_start)"
-        zero_offsets_file="$(arg zero_offsets_file)"/>
+    <xacro:simple_assembly_tracking_ros2_control name="DamiaoArm"/>
 </robot>
