Commit message: update

File: src/simple_assembly_moveit_config/config/simple_assembly_canhat.ros2_control.xacro (robot description, xacro)
@@ -9,72 +9,6 @@
                 <param name="switch_mode_on_activate">true</param>
             </hardware>
-            <!-- Joint 1 (base): Z-type (DM10010), physical top-to-bottom index 7 -->
+            <!-- Joint 1 (base): Z-axis, bottom motor -->
             <joint name="revolute_1_0">
-                <param name="motor_type">DM10010</param>
-                <param name="slave_id">0x03</param>
-                <param name="master_id">0x13</param>
-                <command_interface name="position"/>
-                <command_interface name="velocity"/>
-                <state_interface name="position"/>
-                <state_interface name="velocity"/>
-                <state_interface name="effort"/>
-            </joint>
-            <!-- Joint 2: Y-type (DM4340), physical top-to-bottom index 6 -->
-            <joint name="revolute_2_0">
-                <param name="motor_type">DM4340</param>
-                <param name="slave_id">0x04</param>
-                <param name="master_id">0x14</param>
-                <command_interface name="position"/>
-                <command_interface name="velocity"/>
-                <state_interface name="position"/>
-                <state_interface name="velocity"/>
-                <state_interface name="effort"/>
-            </joint>
-            <!-- Joint 3: Z-type (DM10010), physical top-to-bottom index 5 -->
-            <joint name="revolute_3_0">
-                <param name="motor_type">DM10010</param>
-                <param name="slave_id">0x07</param>
-                <param name="master_id">0x17</param>
-                <command_interface name="position"/>
-                <command_interface name="velocity"/>
-                <state_interface name="position"/>
-                <state_interface name="velocity"/>
-                <state_interface name="effort"/>
-            </joint>
-            <!-- Joint 4: Y-type (DM4340), physical top-to-bottom index 4 -->
-            <joint name="revolute_4_0">
-                <param name="motor_type">DM4340</param>
-                <param name="slave_id">0x06</param>
-                <param name="master_id">0x16</param>
-                <command_interface name="position"/>
-                <command_interface name="velocity"/>
-                <state_interface name="position"/>
-                <state_interface name="velocity"/>
-                <state_interface name="effort"/>
-            </joint>
-            <!-- Joint 5: Z-type (DM10010), physical top-to-bottom index 3 -->
-            <joint name="revolute_5_0">
-                <param name="motor_type">DM10010</param>
-                <param name="slave_id">0x05</param>
-                <param name="master_id">0x15</param>
-                <command_interface name="position"/>
-                <command_interface name="velocity"/>
-                <state_interface name="position"/>
-                <state_interface name="velocity"/>
-                <state_interface name="effort"/>
-            </joint>
-            <!-- Joint 6: Y-type (DM4340), physical top-to-bottom index 2 -->
-            <joint name="revolute_6_0">
-                <param name="motor_type">DM4340</param>
-                <param name="slave_id">0x02</param>
-                <param name="master_id">0x12</param>
-                <command_interface name="position"/>
-                <command_interface name="velocity"/>
-                <state_interface name="position"/>
-                <state_interface name="velocity"/>
-                <state_interface name="effort"/>
-            </joint>
-            <!-- Joint 7 bench CAN HAT motor: currently small DM4340 at 0x01/0x11. -->
-            <joint name="revolute_7_0">
                 <param name="motor_type">DM4340</param>
                 <param name="slave_id">0x01</param>
@@ -86,4 +20,70 @@
                 <state_interface name="effort"/>
             </joint>
+            <!-- Joint 2: Y-axis -->
+            <joint name="revolute_2_0">
+                <param name="motor_type">DM10010</param>
+                <param name="slave_id">0x02</param>
+                <param name="master_id">0x12</param>
+                <command_interface name="position"/>
+                <command_interface name="velocity"/>
+                <state_interface name="position"/>
+                <state_interface name="velocity"/>
+                <state_interface name="effort"/>
+            </joint>
+            <!-- Joint 3: Z-axis -->
+            <joint name="revolute_3_0">
+                <param name="motor_type">DM4340</param>
+                <param name="slave_id">0x03</param>
+                <param name="master_id">0x13</param>
+                <command_interface name="position"/>
+                <command_interface name="velocity"/>
+                <state_interface name="position"/>
+                <state_interface name="velocity"/>
+                <state_interface name="effort"/>
+            </joint>
+            <!-- Joint 4: Y-axis -->
+            <joint name="revolute_4_0">
+                <param name="motor_type">DM10010</param>
+                <param name="slave_id">0x04</param>
+                <param name="master_id">0x14</param>
+                <command_interface name="position"/>
+                <command_interface name="velocity"/>
+                <state_interface name="position"/>
+                <state_interface name="velocity"/>
+                <state_interface name="effort"/>
+            </joint>
+            <!-- Joint 5: Z-axis -->
+            <joint name="revolute_5_0">
+                <param name="motor_type">DM4340</param>
+                <param name="slave_id">0x05</param>
+                <param name="master_id">0x15</param>
+                <command_interface name="position"/>
+                <command_interface name="velocity"/>
+                <state_interface name="position"/>
+                <state_interface name="velocity"/>
+                <state_interface name="effort"/>
+            </joint>
+            <!-- Joint 6: Y-axis -->
+            <joint name="revolute_6_0">
+                <param name="motor_type">DM10010</param>
+                <param name="slave_id">0x06</param>
+                <param name="master_id">0x16</param>
+                <command_interface name="position"/>
+                <command_interface name="velocity"/>
+                <state_interface name="position"/>
+                <state_interface name="velocity"/>
+                <state_interface name="effort"/>
+            </joint>
+            <!-- Joint 7: Z-axis, top motor -->
+            <joint name="revolute_7_0">
+                <param name="motor_type">DM4340</param>
+                <param name="slave_id">0x07</param>
+                <param name="master_id">0x17</param>
+                <command_interface name="position"/>
+                <command_interface name="velocity"/>
+                <state_interface name="position"/>
+                <state_interface name="velocity"/>
+                <state_interface name="effort"/>
+            </joint>
         </ros2_control>
     </xacro:macro>

File: src/simple_assembly_tracking_moveit_config/config/simple_assembly_tracking_canhat.ros2_control.xacro (robot description, xacro)
@@ -9,72 +9,6 @@
                 <param name="switch_mode_on_activate">true</param>
             </hardware>
-            <!-- Joint 1 (base): Z-type (DM10010), physical top-to-bottom index 7 -->
+            <!-- Joint 1 (base): Z-axis, bottom motor -->
             <joint name="revolute_1_0">
-                <param name="motor_type">DM10010</param>
-                <param name="slave_id">0x03</param>
-                <param name="master_id">0x13</param>
-                <command_interface name="position"/>
-                <command_interface name="velocity"/>
-                <state_interface name="position"/>
-                <state_interface name="velocity"/>
-                <state_interface name="effort"/>
-            </joint>
-            <!-- Joint 2: Y-type (DM4340), physical top-to-bottom index 6 -->
-            <joint name="revolute_2_0">
-                <param name="motor_type">DM4340</param>
-                <param name="slave_id">0x04</param>
-                <param name="master_id">0x14</param>
-                <command_interface name="position"/>
-                <command_interface name="velocity"/>
-                <state_interface name="position"/>
-                <state_interface name="velocity"/>
-                <state_interface name="effort"/>
-            </joint>
-            <!-- Joint 3: Z-type (DM10010), physical top-to-bottom index 5 -->
-            <joint name="revolute_3_0">
-                <param name="motor_type">DM10010</param>
-                <param name="slave_id">0x07</param>
-                <param name="master_id">0x17</param>
-                <command_interface name="position"/>
-                <command_interface name="velocity"/>
-                <state_interface name="position"/>
-                <state_interface name="velocity"/>
-                <state_interface name="effort"/>
-            </joint>
-            <!-- Joint 4: Y-type (DM4340), physical top-to-bottom index 4 -->
-            <joint name="revolute_4_0">
-                <param name="motor_type">DM4340</param>
-                <param name="slave_id">0x06</param>
-                <param name="master_id">0x16</param>
-                <command_interface name="position"/>
-                <command_interface name="velocity"/>
-                <state_interface name="position"/>
-                <state_interface name="velocity"/>
-                <state_interface name="effort"/>
-            </joint>
-            <!-- Joint 5: Z-type (DM10010), physical top-to-bottom index 3 -->
-            <joint name="revolute_5_0">
-                <param name="motor_type">DM10010</param>
-                <param name="slave_id">0x05</param>
-                <param name="master_id">0x15</param>
-                <command_interface name="position"/>
-                <command_interface name="velocity"/>
-                <state_interface name="position"/>
-                <state_interface name="velocity"/>
-                <state_interface name="effort"/>
-            </joint>
-            <!-- Joint 6: Y-type (DM4340), physical top-to-bottom index 2 -->
-            <joint name="revolute_6_0">
-                <param name="motor_type">DM4340</param>
-                <param name="slave_id">0x02</param>
-                <param name="master_id">0x12</param>
-                <command_interface name="position"/>
-                <command_interface name="velocity"/>
-                <state_interface name="position"/>
-                <state_interface name="velocity"/>
-                <state_interface name="effort"/>
-            </joint>
-            <!-- Joint 7 bench CAN HAT motor: currently small DM4340 at 0x01/0x11. -->
-            <joint name="revolute_7_0">
                 <param name="motor_type">DM4340</param>
                 <param name="slave_id">0x01</param>
@@ -86,4 +20,70 @@
                 <state_interface name="effort"/>
             </joint>
+            <!-- Joint 2: Y-axis -->
+            <joint name="revolute_2_0">
+                <param name="motor_type">DM10010</param>
+                <param name="slave_id">0x02</param>
+                <param name="master_id">0x12</param>
+                <command_interface name="position"/>
+                <command_interface name="velocity"/>
+                <state_interface name="position"/>
+                <state_interface name="velocity"/>
+                <state_interface name="effort"/>
+            </joint>
+            <!-- Joint 3: Z-axis -->
+            <joint name="revolute_3_0">
+                <param name="motor_type">DM4340</param>
+                <param name="slave_id">0x03</param>
+                <param name="master_id">0x13</param>
+                <command_interface name="position"/>
+                <command_interface name="velocity"/>
+                <state_interface name="position"/>
+                <state_interface name="velocity"/>
+                <state_interface name="effort"/>
+            </joint>
+            <!-- Joint 4: Y-axis -->
+            <joint name="revolute_4_0">
+                <param name="motor_type">DM10010</param>
+                <param name="slave_id">0x04</param>
+                <param name="master_id">0x14</param>
+                <command_interface name="position"/>
+                <command_interface name="velocity"/>
+                <state_interface name="position"/>
+                <state_interface name="velocity"/>
+                <state_interface name="effort"/>
+            </joint>
+            <!-- Joint 5: Z-axis -->
+            <joint name="revolute_5_0">
+                <param name="motor_type">DM4340</param>
+                <param name="slave_id">0x05</param>
+                <param name="master_id">0x15</param>
+                <command_interface name="position"/>
+                <command_interface name="velocity"/>
+                <state_interface name="position"/>
+                <state_interface name="velocity"/>
+                <state_interface name="effort"/>
+            </joint>
+            <!-- Joint 6: Y-axis -->
+            <joint name="revolute_6_0">
+                <param name="motor_type">DM10010</param>
+                <param name="slave_id">0x06</param>
+                <param name="master_id">0x16</param>
+                <command_interface name="position"/>
+                <command_interface name="velocity"/>
+                <state_interface name="position"/>
+                <state_interface name="velocity"/>
+                <state_interface name="effort"/>
+            </joint>
+            <!-- Joint 7: Z-axis, top motor -->
+            <joint name="revolute_7_0">
+                <param name="motor_type">DM4340</param>
+                <param name="slave_id">0x07</param>
+                <param name="master_id">0x17</param>
+                <command_interface name="position"/>
+                <command_interface name="velocity"/>
+                <state_interface name="position"/>
+                <state_interface name="velocity"/>
+                <state_interface name="effort"/>
+            </joint>
         </ros2_control>
     </xacro:macro>
