Commit message: Raise camera_link 53.6 mm above cam_mount_assy
Co-Authored-By: Claude Opus 4.7 <noreply@anthropic.com>

File: src/simple_assembly_tracking/urdf/simple_assembly_tracking.urdf.xacro (robot description, xacro)
@@ -15,5 +15,5 @@
         <parent link="cam_mount_assy__1_"/>
         <child link="camera_link"/>
-        <origin xyz="0 0 0" rpy="0 0 0"/>
+        <origin xyz="0 0 0.0536" rpy="0 0 0"/>
     </joint>
     <link name="camera_optical_frame"/>

Commit message: Offset camera_optical_frame 17 mm to image-right of camera_link
Co-Authored-By: Claude Opus 4.7 <noreply@anthropic.com>

File: src/simple_assembly_tracking/urdf/simple_assembly_tracking.urdf.xacro (robot description, xacro)
@@ -21,5 +21,5 @@
         <parent link="camera_link"/>
         <child link="camera_optical_frame"/>
-        <origin xyz="0 0 0" rpy="0 0 1.5708"/>
+        <origin xyz="0.017 0 0" rpy="0 0 1.5708"/>
     </joint>
 </robot>

Commit message: Camera: drop second box visual, put both offsets on optical frame
The added camera_link box was overlapping the OnShape cam_mount mesh and
showing as a second camera block. camera_link is now a pure frame at the
mount. The 53.6 mm up + 17 mm right offsets live on camera_optical_frame
in its own ROS optical axes (X=right, Y=down, Z=forward).

Co-Authored-By: Claude Opus 4.7 <noreply@anthropic.com>

File: src/simple_assembly_tracking/urdf/simple_assembly_tracking.urdf.xacro (robot description, xacro)
@@ -2,24 +2,19 @@
 <robot xmlns:xacro="http://www.ros.org/wiki/xacro" name="simple_assembly_tracking">
     <xacro:include filename="$(find full_assembly)/urdf/simple_assembly.urdf" />
-    <link name="camera_link">
-        <visual>
-            <geometry>
-                <box size="0.04 0.08 0.03"/>
-            </geometry>
-            <material name="camera_black">
-                <color rgba="0.1 0.1 0.1 1"/>
-            </material>
-        </visual>
-    </link>
+    <!-- Pure frame at the OnShape camera mount; mount mesh already shows the camera body. -->
+    <link name="camera_link"/>
     <joint name="camera_joint" type="fixed">
         <parent link="cam_mount_assy__1_"/>
         <child link="camera_link"/>
-        <origin xyz="0 0 0.0536" rpy="0 0 0"/>
+        <origin xyz="0 0 0" rpy="0 0 0"/>
     </joint>
     <link name="camera_optical_frame"/>
+    <!-- ROS optical convention: X=right, Y=down, Z=forward (looking out the lens).
+         Offsets are the camera-perspective offset of the lens centre from the
+         camera_link/cam_mount frame: 17 mm right, 53.6 mm up. -->
     <joint name="camera_optical_joint" type="fixed">
         <parent link="camera_link"/>
         <child link="camera_optical_frame"/>
-        <origin xyz="0.017 0 0" rpy="0 0 1.5708"/>
+        <origin xyz="0.017 -0.0536 0" rpy="0 0 1.5708"/>
     </joint>
 </robot>

Commit message: Reparent camera_link to part_1_17 (white mount on top), drop +Z offset
Co-Authored-By: Claude Opus 4.7 <noreply@anthropic.com>

File: src/simple_assembly_tracking/urdf/simple_assembly_tracking.urdf.xacro (robot description, xacro)
@@ -2,8 +2,8 @@
 <robot xmlns:xacro="http://www.ros.org/wiki/xacro" name="simple_assembly_tracking">
     <xacro:include filename="$(find full_assembly)/urdf/simple_assembly.urdf" />
-    <!-- Pure frame at the OnShape camera mount; mount mesh already shows the camera body. -->
+    <!-- Camera frame anchored to the small white mount (part_1_17) on top of the mount block. -->
     <link name="camera_link"/>
     <joint name="camera_joint" type="fixed">
-        <parent link="cam_mount_assy__1_"/>
+        <parent link="part_1_17"/>
         <child link="camera_link"/>
         <origin xyz="0 0 0" rpy="0 0 0"/>
@@ -11,10 +11,9 @@
     <link name="camera_optical_frame"/>
     <!-- ROS optical convention: X=right, Y=down, Z=forward (looking out the lens).
-         Offsets are the camera-perspective offset of the lens centre from the
-         camera_link/cam_mount frame: 17 mm right, 53.6 mm up. -->
+         17 mm offset = lens centre is 17 mm right of the mount centre. -->
     <joint name="camera_optical_joint" type="fixed">
         <parent link="camera_link"/>
         <child link="camera_optical_frame"/>
-        <origin xyz="0.017 -0.0536 0" rpy="0 0 1.5708"/>
+        <origin xyz="0.017 0 0" rpy="0 0 1.5708"/>
     </joint>
 </robot>

Commit message: Revert camera parent to cam_mount_assy__1_ (part_1_17 had bad orientation)
Co-Authored-By: Claude Opus 4.7 <noreply@anthropic.com>

File: src/simple_assembly_tracking/urdf/simple_assembly_tracking.urdf.xacro (robot description, xacro)
@@ -2,8 +2,8 @@
 <robot xmlns:xacro="http://www.ros.org/wiki/xacro" name="simple_assembly_tracking">
     <xacro:include filename="$(find full_assembly)/urdf/simple_assembly.urdf" />
-    <!-- Camera frame anchored to the small white mount (part_1_17) on top of the mount block. -->
+    <!-- Pure frame at the OnShape camera mount; mount mesh already shows the camera body. -->
     <link name="camera_link"/>
     <joint name="camera_joint" type="fixed">
-        <parent link="part_1_17"/>
+        <parent link="cam_mount_assy__1_"/>
         <child link="camera_link"/>
         <origin xyz="0 0 0" rpy="0 0 0"/>
