Commit message: update

File: src/simple_assembly_tracking/urdf/simple_assembly_tracking.urdf.xacro (robot description, xacro)
@@ -13,7 +13,7 @@
     </link>
     <joint name="camera_joint" type="fixed">
-        <parent link="root"/>
+        <parent link="wrist_link"/>
         <child link="camera_link"/>
-        <origin xyz="0.4 0.0 0.3" rpy="0 0.5236 0"/>
+        <origin xyz="0 0 0.055" rpy="0 0 0"/>
     </joint>
     <link name="camera_optical_frame"/>

Commit message: Align camera optical axis with wrist z

File: src/simple_assembly_tracking/urdf/simple_assembly_tracking.urdf.xacro (robot description, xacro)
@@ -21,5 +21,5 @@
         <parent link="camera_link"/>
         <child link="camera_optical_frame"/>
-        <origin xyz="0 0 0" rpy="-1.5708 0 -1.5708"/>
+        <origin xyz="0 0 0" rpy="0 0 0"/>
     </joint>
 </robot>

Commit message: Rotate camera optical image axes

File: src/simple_assembly_tracking/urdf/simple_assembly_tracking.urdf.xacro (robot description, xacro)
@@ -21,5 +21,5 @@
         <parent link="camera_link"/>
         <child link="camera_optical_frame"/>
-        <origin xyz="0 0 0" rpy="0 0 0"/>
+        <origin xyz="0 0 0" rpy="0 0 1.5708"/>
     </joint>
 </robot>

Commit message: update

File: src/simple_assembly_tracking/urdf/simple_assembly_tracking.urdf.xacro (robot description, xacro)
@@ -1,5 +1,5 @@
 <?xml version="1.0"?>
 <robot xmlns:xacro="http://www.ros.org/wiki/xacro" name="simple_assembly_tracking">
-    <xacro:include filename="$(find simple_assembly)/urdf/simple_assembly.urdf" />
+    <xacro:include filename="$(find full_assembly)/urdf/simple_assembly.urdf" />
     <link name="camera_link">
         <visual>
@@ -13,7 +13,7 @@
     </link>
     <joint name="camera_joint" type="fixed">
-        <parent link="wrist_link"/>
+        <parent link="cam_mount_assy__1_"/>
         <child link="camera_link"/>
-        <origin xyz="0 0 0.055" rpy="0 0 0"/>
+        <origin xyz="0 0 0" rpy="0 0 0"/>
     </joint>
     <link name="camera_optical_frame"/>

Commit message: Revert camera URDF to last known-good frame

File: src/simple_assembly_tracking/urdf/simple_assembly_tracking.urdf.xacro (robot description, xacro)
@@ -2,6 +2,14 @@
 <robot xmlns:xacro="http://www.ros.org/wiki/xacro" name="simple_assembly_tracking">
     <xacro:include filename="$(find full_assembly)/urdf/simple_assembly.urdf" />
-    <!-- Pure frame at the OnShape camera mount; mount mesh already shows the camera body. -->
-    <link name="camera_link"/>
+    <link name="camera_link">
+        <visual>
+            <geometry>
+                <box size="0.04 0.08 0.03"/>
+            </geometry>
+            <material name="camera_black">
+                <color rgba="0.1 0.1 0.1 1"/>
+            </material>
+        </visual>
+    </link>
     <joint name="camera_joint" type="fixed">
         <parent link="cam_mount_assy__1_"/>
@@ -10,10 +18,8 @@
     </joint>
     <link name="camera_optical_frame"/>
-    <!-- ROS optical convention: X=right, Y=down, Z=forward (looking out the lens).
-         17 mm offset = lens centre is 17 mm right of the mount centre. -->
     <joint name="camera_optical_joint" type="fixed">
         <parent link="camera_link"/>
         <child link="camera_optical_frame"/>
-        <origin xyz="0.017 0 0" rpy="0 0 1.5708"/>
+        <origin xyz="0 0 0" rpy="0 0 1.5708"/>
     </joint>
 </robot>
