Commit message: update

File: src/full_assembly/urdf/simple_assembly.urdf (robot description, URDF)
Before this commit: robot simple_assembly, 21 links, 20 joints
Joints:
- joint revolute_1_0: origin xyz=1.17451e-25 1.72433e-18 0.0565 rpy=2.90763e-21 -7.49958e-22 0.449459 -> xyz=1.17451e-25 1.72433e-18 0.0565 rpy=0 0 0
- joint revolute_2_0: origin xyz=-0.027299 -5.21803e-08 0.0815462 rpy=-1.5708 1.39224 -1.5708 -> xyz=-0.027299 -5.21803e-08 0.0815462 rpy=-1.5708 0 -1.5708
- joint revolute_3_0: origin xyz=-2.92192e-17 0 0.0565 rpy=-9.39199e-15 7.88386e-15 2.26486 -> xyz=-2.92192e-17 0 0.0565 rpy=0 0 0
- joint revolute_4_0: origin xyz=-0.027299 -5.21803e-08 0.0815462 rpy=1.5708 1.22316 1.5708 -> xyz=-0.027299 -5.21803e-08 0.0815462 rpy=1.5708 0 1.5708
- joint revolute_5_0: origin xyz=2.498e-16 1.11022e-16 0.0565 rpy=-1.70523e-15 -3.81186e-15 -1.25895 -> xyz=2.498e-16 1.11022e-16 0.0565 rpy=0 0 0
- joint revolute_6_0: origin xyz=-0.027299 -5.21803e-08 0.0815462 rpy=-1.5708 0.988935 -1.5708 -> xyz=-0.027299 -5.21803e-08 0.0815462 rpy=-1.5708 0 -1.5708
- joint revolute_7_0: origin xyz=5.55112e-17 0 0.0565 rpy=-2.97823e-15 5.96537e-16 -1.59471 -> xyz=5.55112e-17 0 0.0565 rpy=0 0 0

Commit message: update

File: src/full_assembly/urdf/simple_assembly.urdf (robot description, URDF)
Before this commit: robot simple_assembly, 21 links, 20 joints
Joints:
- joint revolute_4_0: origin xyz=-0.027299 -5.21803e-08 0.0815462 rpy=1.5708 0 1.5708 -> xyz=-0.027299 -5.21803e-08 0.0815462 rpy=1.5708 3.14159 1.5708

Commit message: update

File: src/full_assembly/urdf/simple_assembly.urdf (robot description, URDF)
Before this commit: robot simple_assembly, 21 links, 20 joints
Joints:
- joint revolute_7_0: limit lower=-6.28318 upper=6.28318 effort=150.0 velocity=15.71 -> lower=-3.14159 upper=3.14159 effort=150.0 velocity=15.71

Commit message: update

File: src/full_assembly/urdf/simple_assembly.urdf (robot description, URDF)
Before this commit: robot simple_assembly, 21 links, 20 joints
Joints:
- joint revolute_7_0: origin xyz=5.55112e-17 0 0.0565 rpy=0 0 0 -> xyz=5.55112e-17 0 0.0565 rpy=0 0 1.5708

File: src/simple_assembly/urdf/simple_assembly.urdf (robot description, URDF)
Before this commit: robot simple_assembly, 17 links, 16 joints
Joints:
- joint revolute_7_0: origin xyz=0 0 0 rpy=0 0 0 -> xyz=0 0 0 rpy=0 0 1.5708
