Commit message: Correct terra_arm masses with datasheet and weighed values
The Fusion export used default materials, so the 10010 motors, 3200 mAh
packs and slip rings came out as solid steel (27.17 kg total). Rewrite
mass, centre of mass and inertia for the 17 affected links: DM-J10010
1.485 kg and DM-J4340P 0.375 kg from the manuals; weighed 3200 mAh
(218 g) and 5000 mAh (1.52 lb) packs; 10.5 oz slip ring with aluminium
base plate and pin; grippers rebuilt part by part (aluminium housing,
TPU jaws and fingers, steel pins, 3.52 oz servos). New total 14.35 kg.
Wiring and electronics are still not modelled.

scripts/step_reach_sim/apply_measured_masses.py reproduces the change.

Co-Authored-By: Claude Opus 5.5 <noreply@anthropic.com>
Claude-Session: https://claude.ai/code/session_01UZht8P8uWzd5XbdWG5ezN3

File: src/terra_arm_description/urdf/arm.urdf (robot description, URDF)
Before this commit: robot terra_arm, 38 links, 37 joints
Links:
- link DM-J10010L-2EC_Motor_1: mass 3.92262518 -> 1.485
- link DM-J10010L-2EC_Motor_2: mass 3.92262518 -> 1.485
- link DM-J10010L-2EC_Motor_3: mass 3.92262518 -> 1.485
- link DM-J4340P-2EC_Motor_1: mass 0.386823391 -> 0.375
- link DM-J4340P-2EC_Motor_2: mass 0.386823391 -> 0.375
- link DM-J4340P-2EC_Motor_3: mass 0.386823391 -> 0.375
- link DM-J4340P-2EC_Motor_4: mass 0.386823391 -> 0.375
- link EndEffectorAssembly_v3_1: mass 1.36223202 -> 0.911573759
- link EndEffectorAssembly_v3_2: mass 1.36223202 -> 0.911573759
- link LiPo_3200mAh_batt_3: mass 0.75831 -> 0.218
- link LiPo_3200mAh_batt_4: mass 0.75831 -> 0.218
- link LiPo_5000mAh_Batt_2: mass 0.67662868 -> 0.689460402
- link LiPo_5000mAh_Batt_3: mass 0.67662868 -> 0.689460402
- link SlipRing_1_rotor: mass 0.13463513 -> 0.115269516
- link SlipRing_1_stator: mass 2.10570352 -> 0.373786227
- link SlipRing_2_rotor: mass 0.13463513 -> 0.115269516
- link SlipRing_2_stator: mass 2.10570352 -> 0.373786227
